Commit message: Lots of progress, model is working and accurate, starting launch file

File: src/jrobot.urdf (robot description, URDF)
Before this commit: robot jrobot, 5 links, 4 joints
Links:
- link base: geometry collision box size=0.94 0.78 1.90; visual box size=0.94 0.78 1.90
Joints:
- joint base_laser_horiz_joint: origin xyz=0.2325 0.0001 1.9201 rpy=0.2325 -0.0001 1.9201 -> xyz=0. 0.000 0.0
- joint base_laser_vert_bottom_joint: origin xyz=0.3158 -0.0021 0.5100 rpy=3.1355 -1.3045 0.0025 -> xyz=0 0 0.092
- joint base_laser_vert_top_left_joint: origin xyz=0.2997 0.1531 1.8443 rpy=1.1780 0.6198 1.9560 -> (none)
- joint base_laser_vert_top_right_joint: origin xyz=0.2978 -0.1450 1.8451 rpy=-1.1760 0.6313 -1.9377 -> xyz=0 0 0
