Commit message: Added to URDF, created XACRO, updated launch file

File: urdf/robot.xacro (robot description, xacro)
@@ -1,3 +1,4 @@
-<robot name="jrobot">
+<?xml version="1.0"?>
+<robot xmlns:xacro="http://www.ros.org/wiki/xacro" name="jrobot">
 	<link name="base">
 		<visual>
@@ -85,21 +86,23 @@
 		</collision>
 	</link>
-	<link name="wheel_left">
-		<visual>
-			<origin xyz="-0.1 0.4 0" rpy="-1.5707 0 0" />
-			<geometry>
-				<cylinder radius="0.2" length="0.05" />
-			</geometry>
-			<material name="Cyan">
-			<color rgba="0 1.0 1.0 1.0"/>
-			</material>
-      		</visual>
-		<collision>
-			<origin xyz="-0.1 0.4 0" rpy="-1.5707 0 0" />
-			<geometry>
-				<cylinder radius="0.2" length="0.05" />
-			</geometry>
-		</collision>
-	</link>
+	<xacro:macro name="xacro_name" params="suffix reflect">
+		<link name="wheel_${suffix}">
+			<visual>
+				<origin xyz="-0.1 0.4 0" rpy="-1.5707 0 0" />
+				<geometry>
+					<cylinder radius="0.2" length="0.05" />
+				</geometry>
+				<material name="Cyan">
+				<color rgba="0 1.0 1.0 1.0"/>
+				</material>
+	      		</visual>
+			<collision>
+				<origin xyz="-0.1 0.4 0" rpy="-1.5707 0 0" />
+				<geometry>
+					<cylinder radius="0.2" length="0.05" />
+				</geometry>
+			</collision>
+		</link>
+	</xacro:macro>
 	<link name="wheel_center">
 		<visual>
@@ -146,11 +149,13 @@
 		<!-- <limit effort="30" velocity="1.0" lower="-2.2" upper="0.7" /> -->
 	</joint>
-	<joint name="base_wheel_left_joint" type="fixed">
-		<!-- <origin xyz="0.2325 0.0001 1.9201" rpy="0.2325 -0.0001 1.9201" /> -->
-		<origin xyz="0. 0.000 0.0"/>
-		<parent link="base"/>
-		<child link="wheel_left"/>
-		<!-- <limit effort="30" velocity="1.0" lower="-2.2" upper="0.7" /> -->
-	</joint>
+	<xacro:macro name="xacro_name" params="suffix reflect">
+		<joint name="base_wheel_${suffix}_joint" type="fixed">
+			<!-- <origin xyz="0.2325 0.0001 1.9201" rpy="0.2325 -0.0001 1.9201" /> -->
+			<origin xyz="0. 0.000 0.0"/>
+			<parent link="base"/>
+			<child link="wheel_${suffix}"/>
+			<!-- <limit effort="30" velocity="1.0" lower="-2.2" upper="0.7" /> -->
+		</joint>
+	</xacro:macro>
 	<joint name="base_wheel_center_joint" type="fixed">
 		<!-- <origin xyz="0.2325 0.0001 1.9201" rpy="0.2325 -0.0001 1.9201" /> -->
@@ -160,3 +165,4 @@
 		<!-- <limit effort="30" velocity="1.0" lower="-2.2" upper="0.7" /> -->
 	</joint>
+	 <xacro:xacro_name suffix="leftL" reflect="1" />
 </robot>

Commit message: Working XACRO for wheels and launch file is updated.

File: urdf/robot.xacro (robot description, xacro)
@@ -89,5 +89,6 @@
 		<link name="wheel_${suffix}">
 			<visual>
-				<origin xyz="-0.1 0.4 0" rpy="-1.5707 0 0" />
+				<origin xyz="-0.1 ${reflect * 0.4} 0" rpy="-1.5707 0 0"/>
+				<!-- <origin xyz="-0.1 0.4 0" rpy="-1.5707 0 0" /> -->
 				<geometry>
 					<cylinder radius="0.2" length="0.05" />
@@ -98,5 +99,6 @@
 	      		</visual>
 			<collision>
-				<origin xyz="-0.1 0.4 0" rpy="-1.5707 0 0" />
+				<origin xyz="-0.1 ${reflect * 0.4} 0" rpy="-1.5707 0 0"/>
+				<!-- <origin xyz="-0.1 0.4 0" rpy="-1.5707 0 0" /> -->
 				<geometry>
 					<cylinder radius="0.2" length="0.05" />
@@ -105,4 +107,6 @@
 		</link>
 	</xacro:macro>
+	<xacro:xacro_name suffix="left" reflect="1" />
+	<xacro:xacro_name suffix="right" reflect="-1" />
 	<link name="wheel_center">
 		<visual>
@@ -165,4 +169,5 @@
 		<!-- <limit effort="30" velocity="1.0" lower="-2.2" upper="0.7" /> -->
 	</joint>
-	 <xacro:xacro_name suffix="leftL" reflect="1" />
+	 <xacro:xacro_name suffix="left" reflect="1" />
+	 <xacro:xacro_name suffix="right" reflect="-1" />
 </robot>

Commit message: kept working on xacro with revolutions

File: urdf/robot.xacro (robot description, xacro)
@@ -154,18 +154,20 @@
 	</joint>
 	<xacro:macro name="xacro_name" params="suffix reflect">
-		<joint name="base_wheel_${suffix}_joint" type="fixed">
+		<joint name="base_wheel_${suffix}_joint" type="continuous">
 			<!-- <origin xyz="0.2325 0.0001 1.9201" rpy="0.2325 -0.0001 1.9201" /> -->
-			<origin xyz="0. 0.000 0.0"/>
+			<origin xyz="0. 0 0.0"/>
+			<axis xyz="0 0.1 0" />
 			<parent link="base"/>
 			<child link="wheel_${suffix}"/>
-			<!-- <limit effort="30" velocity="1.0" lower="-2.2" upper="0.7" /> -->
+			<limit effort="30" velocity="1.0" lower="-2.2" upper="0.7" />
 		</joint>
 	</xacro:macro>
-	<joint name="base_wheel_center_joint" type="fixed">
+	<joint name="base_wheel_center_joint" type="continuous">
 		<!-- <origin xyz="0.2325 0.0001 1.9201" rpy="0.2325 -0.0001 1.9201" /> -->
 		<origin xyz="0. 0.000 0.0"/>
+		<axis xyz="0 0.9 0"/>
 		<parent link="base"/>
 		<child link="wheel_center"/>
-		<!-- <limit effort="30" velocity="1.0" lower="-2.2" upper="0.7" /> -->
+		<limit effort="30" velocity="1.0" lower="-2.2" upper="0.7" />
 	</joint>
 	 <xacro:xacro_name suffix="left" reflect="1" />

Commit message: Finished the xacro and updated some features. Also creates a read me file.

File: urdf/robot.xacro (robot description, xacro)
@@ -18,5 +18,7 @@
 		</collision>
 	</link>
-	<link name="laser_vert_bottom">
+	<xacro:include filename="$(find gazebo_plugins)/test/multi_robot_scenario/xacro/laser/hokuyo.xacro" />
+	<xacro:laser name="laser_vert_bottom" parent="base" xyz="0.3157894464801903 -0.002068548615034871 0.5099999434059285" rpy="3.1354753 -1.3045001 0.0024658" meshes="package://gazebo_plugins/test/multi_robot_scenario/meshes/laser" />
+	<!-- <link name="laser_vert_bottom">
 		<visual>
 			<origin xyz="0.3158 -0.0021 0.5100" rpy="3.1355 -1.3045 0.0025" />
@@ -34,5 +36,5 @@
 			</geometry>
 		</collision>
-	</link>
+	</link> -->
 	<link name="laser_vert_top_right">
 		<visual>
@@ -69,4 +71,10 @@
 		</collision>
 	</link>
+	<xacro:include filename="$(find velodyne_description)/urdf/VLP-16.urdf.xacro"/>
+	<!-- Invoke the macro to define the Hokuyo LIDAR.-->
+	<VLP-16 parent="base" name="laser_horiz" topic="laser_horiz/packets" hz="10" samples="440" gpu="false">
+		<origin xyz="0.2325416305773505 -0.0001380069427607134 1.920122926231907" rpy="-0.0012068 0.114646 -0.0015308" />
+	</VLP-16>
+	<!--
 	<link name="laser_horiz">
 		<visual>
@@ -85,5 +93,5 @@
 			</geometry>
 		</collision>
-	</link>
+	</link> -->
 	<xacro:macro name="xacro_name" params="suffix reflect">
 		<link name="wheel_${suffix}">
@@ -126,11 +134,11 @@
 		</collision>
 	</link>
-	<joint name="base_laser_vert_bottom_joint" type="fixed">
-		<!-- <origin xyz="0.3158 -0.0021 0.5100" rpy="3.1355 -1.3045 0.0025" /> -->
+<!-- 	<joint name="base_laser_vert_bottom_joint" type="fixed">
+		//<origin xyz="0.3158 -0.0021 0.5100" rpy="3.1355 -1.3045 0.0025" />
 		<origin xyz="0 0 0.092" />
 		<parent link="base"/>
 		<child link="laser_vert_bottom"/>
-		<!-- <limit effort="30" velocity="1.0" lower="-2.2" upper="0.7" /> -->
-	</joint>
+		// <limit effort="30" velocity="1.0" lower="-2.2" upper="0.7" />
+	</joint> -->
 	<joint name="base_laser_vert_top_right_joint" type="fixed">
 		<!-- <origin xyz="0.2978 -0.1450 1.8451" rpy="-1.1760 0.6313 -1.9377" /> -->

Commit message: Added new launch file and updated xacro

File: urdf/robot.xacro (robot description, xacro)
@@ -1,183 +1,27 @@
 <?xml version="1.0"?>
-<robot xmlns:xacro="http://www.ros.org/wiki/xacro" name="jrobot">
-	<link name="base">
+<robo xmlns:xacro="http://www.ros.org/wiki/xacro" name="navvis_m6">
+	<xacro:include filename="$(find RobotDesc)/urdf/robotLab4.xacro" />
+	<link name="base_link" />
+	<joint name="base_link_base_joint" type="fixed">
+		<parent link="base_link" />
+		<child link="base" />
+		<origin xyz="0.07 0 1.792" rpy="0.0 ${pi} 0.0" />
+	</joint>
+	<joint name="base_link_imu_joint" type="fixed">
+		<parent link="base_link" />
+		<child link="imu" />
+		<origin xyz="0.0 0.0 0.0" rpy="3.1405788 0.0034281 3.1382064" />
+	</joint>
+	<link name="imu">
 		<visual>
-			<origin xyz="-0.2 0 0.95" rpy="0 0 0" />
 			<geometry>
-				<box size="0.94 0.78 1.90" />
+				<sphere adius="0.1" />
 			</geometry>
-			<material name="Cyan">
-			<color rgba="0 1.0 1.0 1.0"/>
-			</material>
-      		</visual>
+		</visual>
 		<collision>
-			<origin xyz="-0.5 0 0.95" rpy="0 0 0"/>
 			<geometry>
-				<box size="0.94 0.78 1.90" />
+				<sphere radius="0.1" />
 			</geometry>
 		</collision>
 	</link>
-	<xacro:include filename="$(find gazebo_plugins)/test/multi_robot_scenario/xacro/laser/hokuyo.xacro" />
-	<xacro:laser name="laser_vert_bottom" parent="base" xyz="0.3157894464801903 -0.002068548615034871 0.5099999434059285" rpy="3.1354753 -1.3045001 0.0024658" meshes="package://gazebo_plugins/test/multi_robot_scenario/meshes/laser" />
-	<!-- <link name="laser_vert_bottom">
-		<visual>
-			<origin xyz="0.3158 -0.0021 0.5100" rpy="3.1355 -1.3045 0.0025" />
-			<geometry>
-				<box size="0.062 0.062 0.087" />
-			</geometry>
-			<material name="Cyan">
-			<color rgba="0 1.0 1.0 1.0"/>
-			</material>
-      		</visual>
-		<collision>
-			<origin xyz="0.2325 0.0001 1.9201" rpy="3.1355 -1.3045 0.0025" />
-			<geometry>
-				<box size="0.062 0.062 0.087" />
-			</geometry>
-		</collision>
-	</link> -->
-	<link name="laser_vert_top_right">
-		<visual>
-			<origin xyz="0.2978 -0.1450 1.8451" rpy="-1.1760 0.6313 -1.9377" />
-			<geometry>
-				<box size="0.062 0.062 0.087" />
-			</geometry>
-			<material name="Cyan">
-			<color rgba="0 1.0 1.0 1.0"/>
-			</material>
-      		</visual>
-		<collision>
-			<origin xyz="0.2978 -0.1450 1.8451" rpy="-1.1760 0.6313 -1.9377" />
-			<geometry>
-				<box size="0.062 0.062 0.087" />
-			</geometry>
-		</collision>
-	</link>
-	<link name="laser_vert_top_left">
-		<visual>
-			<origin xyz="0.2997 0.1531 1.8443" rpy="1.1780 0.6198 1.9560" />
-			<geometry>
-				<box size="0.062 0.062 0.087" />
-			</geometry>
-			<material name="Cyan">
-			<color rgba="0 1.0 1.0 1.0"/>
-			</material>
-      		</visual>
-		<collision>
-			<origin xyz="0.2978 -0.1450 1.8451" rpy="1.1780 0.6198 1.9560" />
-			<geometry>
-				<box size="0.062 0.062 0.087" />
-			</geometry>
-		</collision>
-	</link>
-	<xacro:include filename="$(find velodyne_description)/urdf/VLP-16.urdf.xacro"/>
-	<!-- Invoke the macro to define the Hokuyo LIDAR.-->
-	<VLP-16 parent="base" name="laser_horiz" topic="laser_horiz/packets" hz="10" samples="440" gpu="false">
-		<origin xyz="0.2325416305773505 -0.0001380069427607134 1.920122926231907" rpy="-0.0012068 0.114646 -0.0015308" />
-	</VLP-16>
-	<!--
-	<link name="laser_horiz">
-		<visual>
-			<origin xyz="0.2325 0.0001 1.9201" rpy="0.2325 -0.0001 1.9201" />
-			<geometry>
-				<cylinder radius="0.052" length="0.072" />
-			</geometry>
-			<material name="Cyan">
-			<color rgba="0 1.0 1.0 1.0"/>
-			</material>
-      		</visual>
-		<collision>
-			<origin xyz="0.2325 0.0001 1.9201" rpy="0.2325 -0.0001 1.9201" />
-			<geometry>
-				<cylinder radius="0.052" length="0.072" />
-			</geometry>
-		</collision>
-	</link> -->
-	<xacro:macro name="xacro_name" params="suffix reflect">
-		<link name="wheel_${suffix}">
-			<visual>
-				<origin xyz="-0.1 ${reflect * 0.4} 0" rpy="-1.5707 0 0"/>
-				<!-- <origin xyz="-0.1 0.4 0" rpy="-1.5707 0 0" /> -->
-				<geometry>
-					<cylinder radius="0.2" length="0.05" />
-				</geometry>
-				<material name="Cyan">
-				<color rgba="0 1.0 1.0 1.0"/>
-				</material>
-	      		</visual>
-			<collision>
-				<origin xyz="-0.1 ${reflect * 0.4} 0" rpy="-1.5707 0 0"/>
-				<!-- <origin xyz="-0.1 0.4 0" rpy="-1.5707 0 0" /> -->
-				<geometry>
-					<cylinder radius="0.2" length="0.05" />
-				</geometry>
-			</collision>
-		</link>
-	</xacro:macro>
-	<xacro:xacro_name suffix="left" reflect="1" />
-	<xacro:xacro_name suffix="right" reflect="-1" />
-	<link name="wheel_center">
-		<visual>
-			<origin xyz="0 0.1 0" rpy="-1.5707 0 0" />
-			<geometry>
-				<cylinder radius="0.15" length="0.05" />
-			</geometry>
-			<material name="Cyan">
-			<color rgba="0 1.0 1.0 1.0"/>
-			</material>
-      		</visual>
-		<collision>
-			<origin xyz="0 0.1 0" rpy="-1.5707 0 0" />
-			<geometry>
-				<cylinder radius="0.15" length="0.05" />
-			</geometry>
-		</collision>
-	</link>
-<!-- 	<joint name="base_laser_vert_bottom_joint" type="fixed">
-		//<origin xyz="0.3158 -0.0021 0.5100" rpy="3.1355 -1.3045 0.0025" />
-		<origin xyz="0 0 0.092" />
-		<parent link="base"/>
-		<child link="laser_vert_bottom"/>
-		// <limit effort="30" velocity="1.0" lower="-2.2" upper="0.7" />
-	</joint> -->
-	<joint name="base_laser_vert_top_right_joint" type="fixed">
-		<!-- <origin xyz="0.2978 -0.1450 1.8451" rpy="-1.1760 0.6313 -1.9377" /> -->
-		<origin xyz="0 0 0" />
-		<parent link="base"/>
-		<child link="laser_vert_top_right"/>
-		<!-- <limit effort="30" velocity="1.0" lower="-2.2" upper="0.7" /> -->
-	</joint>
-	<joint name="base_laser_vert_top_left_joint" type="fixed">
-		<!-- <origin xyz="0.2997 0.1531 1.8443" rpy="1.1780 0.6198 1.9560" /> -->
-		<parent link="base"/>
-		<child link="laser_vert_top_left"/>
-		<!-- <limit effort="30" velocity="1.0" lower="-2.2" upper="0.7" /> -->
-	</joint>
-	<joint name="base_laser_horiz_joint" type="fixed">
-		<!-- <origin xyz="0.2325 0.0001 1.9201" rpy="0.2325 -0.0001 1.9201" /> -->
-		<origin xyz="0. 0.000 0.0"/>
-		<parent link="base"/>
-		<child link="laser_horiz"/>
-		<!-- <limit effort="30" velocity="1.0" lower="-2.2" upper="0.7" /> -->
-	</joint>
-	<xacro:macro name="xacro_name" params="suffix reflect">
-		<joint name="base_wheel_${suffix}_joint" type="continuous">
-			<!-- <origin xyz="0.2325 0.0001 1.9201" rpy="0.2325 -0.0001 1.9201" /> -->
-			<origin xyz="0. 0 0.0"/>
-			<axis xyz="0 0.1 0" />
-			<parent link="base"/>
-			<child link="wheel_${suffix}"/>
-			<limit effort="30" velocity="1.0" lower="-2.2" upper="0.7" />
-		</joint>
-	</xacro:macro>
-	<joint name="base_wheel_center_joint" type="continuous">
-		<!-- <origin xyz="0.2325 0.0001 1.9201" rpy="0.2325 -0.0001 1.9201" /> -->
-		<origin xyz="0. 0.000 0.0"/>
-		<axis xyz="0 0.9 0"/>
-		<parent link="base"/>
-		<child link="wheel_center"/>
-		<limit effort="30" velocity="1.0" lower="-2.2" upper="0.7" />
-	</joint>
-	 <xacro:xacro_name suffix="left" reflect="1" />
-	 <xacro:xacro_name suffix="right" reflect="-1" />
 </robot>

Commit message: Working status with trails, updated ream me and some configurations.

File: urdf/robot.xacro (robot description, xacro)
@@ -16,5 +16,5 @@
 		<visual>
 			<geometry>
-				<sphere adius="0.1" />
+				<sphere radius="0.1" />
 			</geometry>
 		</visual>
